Commit message: TCP changed

File: EasyRobot/easyrobot/urdf/easyrobot.urdf (robot description, URDF)
Before this commit: robot easyrobot, 5 links, 4 joints
Joints:
- joint link2ToTCP: origin xyz=0 0 0.425 rpy=0 0 1.57 -> xyz=0 0 0.475 rpy=0 0 1.57

Commit message: Added dummy inertials

File: EasyRobot/easyrobot/urdf/easyrobot.urdf (robot description, URDF)
Before this commit: robot easyrobot, 5 links, 4 joints
Links:
- link base: mass None -> 1; geometry collision box size=0.5 0.05 0.1; visual box size=0.5 0.05 0.1
- link link1: mass None -> 1; geometry collision box size=0.5 0.05 0.1; visual box size=0.5 0.05 0.1
- link link2: mass None -> 1; geometry collision box size=0.5 0.05 0.1; visual box size=0.5 0.05 0.1
