Commit message: GZ_SIM

File: EasyRobot/easyrobot/urdf/gzbot.urdf (robot description, URDF)
Before this commit: robot easyrobot, 5 links, 4 joints
Links:
- link base: mass 1 -> 10
- link link1: mass 1 -> 5
- link link2: mass 1 -> 5
Joints:
- joint fixedFrameToWorld: origin xyz=0 0 0.5 rpy=0 0 0 -> xyz=0 0 1 rpy=0 0 0
- joint joint1: limit lower=-3.141 upper=3.141 effort=0 velocity=1 -> lower=-61.2831 upper=61.2831 effort=1000 velocity=1000; origin xyz=0 0.05 0.45 rpy=0 0 0 -> xyz=0 0.05 0.45 rpy=0 0.053 0
- joint joint2: limit lower=-3.141 upper=3.141 effort=0 velocity=1 -> lower=-61.2831 upper=61.2831 effort=1000 velocity=1000; origin xyz=0 0.05 0.45 rpy=0 0 0 -> xyz=0 0.05 0.45 rpy=0 0.056 0

Commit message: Joint Sate Publisher Plugin corrected

File: EasyRobot/easyrobot/urdf/gzbot.urdf (robot description, URDF)
Before this commit: robot easyrobot, 5 links, 4 joints
Joints:
- joint joint1: limit lower=-61.2831 upper=61.2831 effort=1000 velocity=1000 -> lower=-6.2831 upper=6.2831 effort=1000 velocity=1000
- joint joint2: limit lower=-61.2831 upper=61.2831 effort=1000 velocity=1000 -> lower=-6.2831 upper=6.2831 effort=1000 velocity=1000

Commit message: A lot of bug fixing

File: EasyRobot/easyrobot/urdf/gzbot.urdf (robot description, URDF)
Before this commit: robot easyrobot, 5 links, 4 joints
Links:
- link base: mass 10 -> 10.0
- link link1: mass 5 -> 5.0
- link link2: mass 5 -> 5.0
Joints:
- joint fixedFrameToWorld: origin xyz=0 0 1 rpy=0 0 0 -> xyz=0.0 0.0 1.0 rpy=0.0 0.0 0.0
- joint joint1: limit lower=-6.2831 upper=6.2831 effort=1000 velocity=1000 -> lower=-6.2831 upper=6.2831 effort=100.0 velocity=10.0; origin xyz=0 0.05 0.45 rpy=0 0.053 0 -> xyz=0.0 0.05 0.45 rpy=0.0 0.0 0.0
- joint joint2: limit lower=-6.2831 upper=6.2831 effort=1000 velocity=1000 -> lower=-6.2831 upper=6.2831 effort=100.0 velocity=10.0; origin xyz=0 0.05 0.45 rpy=0 0.056 0 -> xyz=0.0 0.05 0.45 rpy=0.0 0.0 0.0
- joint link2ToTCP: origin xyz=0 0 0.475 rpy=0 0 1.57 -> xyz=0.0 0.0 0.475 rpy=0.0 0.0 1.57

Commit message: New Moveit Launch file

File: EasyRobot/easyrobot/urdf/gzbot.urdf (robot description, URDF)
Before this commit: robot easyrobot, 5 links, 4 joints
Joints:
- joint joint1: limit lower=-6.2831 upper=6.2831 effort=100.0 velocity=10.0 -> lower=-6.2831 upper=6.2831 effort=200.0 velocity=10.0

File: EasyRobot/moveit_easyrobot/config/easyrobot.urdf.xacro (robot description, xacro)
@@ -4,6 +4,6 @@
     <!-- Import easyrobot urdf file -->
     <xacro:include filename="$(find easyrobot)/urdf/gzbot.urdf" />
-    <!-- Import control_xacro -->
+    <!-- Import control_xacro
     <xacro:include filename="easyrobot.ros2_control.xacro" />
-    <xacro:easyrobot_ros2_control name="FakeSystem" initial_positions_file="$(arg initial_positions_file)"/>
+    <xacro:easyrobot_ros2_control name="FakeSystem" initial_positions_file="$(arg initial_positions_file)"/>-->
 </robot>
