Commit message: gz support added

File: install/easyrobot/share/easyrobot/urdf/easyrobot.urdf (robot description, URDF)
Before this commit: robot easyrobot, 5 links, 4 joints
Links:
- removed link world
- added link fixedFrame
- link base: mass 10 -> 1
- link link1: mass 5 -> 1
- link link2: mass 5 -> 1
Joints:
- joint fixedFrameToWorld: origin xyz=0 0 1 rpy=0 0 0 -> xyz=0 0 0.5 rpy=0 0 0; parent world -> fixedFrame
- joint joint1: limit lower=-61.2831 upper=61.2831 effort=1000 velocity=1000 -> lower=-3.141 upper=3.141 effort=1000 velocity=1000; origin xyz=0 0.05 0.45 rpy=0 0.053 0 -> xyz=0 0.05 0.45 rpy=0 0 0
- joint joint2: limit lower=-61.2831 upper=61.2831 effort=1000 velocity=1000 -> lower=-3.141 upper=3.141 effort=1000 velocity=1000; origin xyz=0 0.05 0.45 rpy=0 0.056 0 -> xyz=0 0.05 0.45 rpy=0 0 0
